File: 4-port-hub/4-port-hub.kicad_pcb (KiCad board)
At the start: 2 copper layers, 40.6 x 38.1 mm, 12 parts, among them J1 USB_A_Stacked, J2 USB_A_Stacked, J3 Conn_01x04_Pin, U1 SL2.1A, Y1 Crystal

Commit message: Improve signal routes
Parts:
- moved Y1 2.54 mm to (132.8, 88.2)
- moved C1 0.92 mm to (144.3, 84.3)
- moved C2 0.92 mm to (146.3, 84.3)
- moved C3 0.57 mm to (149.4, 84.3)
- turned C4 to 180 degrees
- turned C6 to 180 degrees
- turned C7 to 180 degrees
Routing:
- net +5V: track 84.2 -> 95.1 mm, vias 4 -> 0
- net Net-(U1-XIN): track 9.71 -> 12.2 mm
- net Net-(U1-XOUT): track 11.5 -> 14.0 mm
- net Net-(U1-VDD3): track 3.48 -> 2.97 mm
- net GND: track 0.00 -> 0.11 mm, vias 6 -> 8
